File: hardware/sca.brd (EAGLE design)
At the start: 160 x 100 mm, 30 parts

Commit message: added frame and cleaned up
Connections:
- removed net N$6 (its old number): JP2.2
- removed net SDO/ADR: JP2.5
Changed lines of the file:
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@@
 <contactref element="R19" pad="2"/>
 <contactref element="JP4" pad="3"/>
+<contactref element="R2" pad="2"/>
+<contactref element="U$1" pad="GND"/>
 <contactref element="LED1" pad="K"/>
 <contactref element="LED2" pad="K"/>
 <contactref element="LED3" pad="K"/>
-<contactref element="R2" pad="2"/>
-<contactref element="U$1" pad="GND"/>
 <wire x1="-83.82" y1="-31.75" x2="-76.2" y2="-44.45" width="0" layer="19" extent="1-1"/>
 <wire x1="-83.82" y1="-26.67" x2="-83.82" y2="-31.75" width="0" layer="19" extent="1-1"/>
@@
 <contactref element="JP4" pad="1"/>
 <wire x1="62.23" y1="33.147" x2="62.23" y2="32.512" width="0.254" layer="16"/>
-</signal>
-<signal name="N$2">
-<contactref element="XB1" pad="2"/>
-<contactref element="U$1" pad="0/RX"/>
-<wire x1="-36.4" y1="27.32" x2="-71.12" y2="58.42" width="0" layer="19" extent="1-1"/>
 </signal>
 <signal name="N$4">
@@
 <contactref element="5V_REG" pad="1"/>
 <contactref element="C10" pad="1"/>
+<contactref element="R1" pad="2"/>
 <contactref element="R20" pad="1"/>
-<contactref element="R1" pad="2"/>
 <wire x1="-64.77" y1="2.54" x2="-76.2" y2="-38.1" width="0" layer="19" extent="1-1"/>
 <wire x1="-80.01" y1="80.01" x2="-64.77" y2="2.54" width="0" layer="19" extent="1-1"/>
 <wire x1="-57.15" y1="93.98" x2="-80.01" y2="80.01" width="0" layer="19" extent="1-1"/>
-</signal>
-<signal name="N$5">
-<contactref element="U$1" pad="14/A0"/>
-<contactref element="PH1" pad="2"/>
-<contactref element="R12" pad="2"/>
-<wire x1="-43.18" y1="73.66" x2="-40.21" y2="81.28" width="0" layer="19" extent="1-1"/>
-<wire x1="-59.69" y1="95.25" x2="-40.21" y2="81.28" width="0" layer="19" extent="1-1"/>
-</signal>
-<signal name="N$10">
-<contactref element="PH2" pad="2"/>
-<contactref element="R13" pad="2"/>
-<contactref element="U$1" pad="15/A1"/>
-<wire x1="-45.72" y1="73.66" x2="-50.37" y2="81.28" width="0" layer="19" extent="1-1"/>
-<wire x1="-64.77" y1="95.25" x2="-50.37" y2="81.28" width="0" layer="19" extent="1-1"/>
-</signal>
-<signal name="N$11">
-<contactref element="PH3" pad="2"/>
-<contactref element="R14" pad="2"/>
-<contactref element="U$1" pad="16/A2"/>
-<wire x1="-60.53" y1="81.28" x2="-69.85" y2="95.25" width="0" layer="19" extent="1-1"/>
-<wire x1="-48.26" y1="73.66" x2="-60.53" y2="81.28" width="0" layer="19" extent="1-1"/>
-</signal>
-<signal name="N$12">
-<contactref element="PH4" pad="2"/>
-<contactref element="R15" pad="2"/>
-<contactref element="U$1" pad="17/A3"/>
-<wire x1="-70.69" y1="81.28" x2="-50.8" y2="73.66" width="0" layer="19" extent="1-1"/>
-<wire x1="-74.93" y1="95.25" x2="-70.69" y2="81.28" width="0" layer="19" extent="1-1"/>
-</signal>
-<signal name="SDO/ADR">
-<contactref element="JP2" pad="5"/>
 </signal>
 <signal name="CS">
@@
 <wire x1="-55.88" y1="73.66" x2="23.495" y2="6.35" width="0" layer="19" extent="1-1"/>
 </signal>
-<signal name="N$6">
-<contactref element="JP2" pad="2"/>
-</signal>
 <signal name="N$3">
 <contactref element="JP4" pad="9"/>
@@
 <wire x1="-66.04" y1="58.42" x2="-86.36" y2="-38.1" width="0" layer="19" extent="1-1"/>
 </signal>
+<signal name="N$1">
+<contactref element="XB1" pad="2"/>
+<contactref element="U$1" pad="0/RX"/>
+<wire x1="-36.4" y1="27.32" x2="-71.12" y2="58.42" width="0" layer="19" extent="1-1"/>
+</signal>
+<signal name="N$2">
+<contactref element="PH2" pad="2"/>
+<contactref element="R13" pad="2"/>
+<contactref element="U$1" pad="15/A1"/>
+<wire x1="-45.72" y1="73.66" x2="-50.37" y2="81.28" width="0" layer="19" extent="1-1"/>
+<wire x1="-64.77" y1="95.25" x2="-50.37" y2="81.28" width="0" layer="19" extent="1-1"/>
+</signal>
+<signal name="N$6">
+<contactref element="PH1" pad="2"/>
+<contactref element="R12" pad="2"/>
+<contactref element="U$1" pad="14/A0"/>
+<wire x1="-43.18" y1="73.66" x2="-40.21" y2="81.28" width="0" layer="19" extent="1-1"/>
+<wire x1="-59.69" y1="95.25" x2="-40.21" y2="81.28" width="0" layer="19" extent="1-1"/>
+</signal>
+<signal name="N$15">
+<contactref element="PH3" pad="2"/>
+<contactref element="R14" pad="2"/>
+<contactref element="U$1" pad="16/A2"/>
+<wire x1="-60.53" y1="81.28" x2="-69.85" y2="95.25" width="0" layer="19" extent="1-1"/>
+<wire x1="-48.26" y1="73.66" x2="-60.53" y2="81.28" width="0" layer="19" extent="1-1"/>
+</signal>
+<signal name="N$19">
+<contactref element="PH4" pad="2"/>
+<contactref element="R15" pad="2"/>
+<contactref element="U$1" pad="17/A3"/>
+<wire x1="-70.69" y1="81.28" x2="-50.8" y2="73.66" width="0" layer="19" extent="1-1"/>
+<wire x1="-74.93" y1="95.25" x2="-70.69" y2="81.28" width="0" layer="19" extent="1-1"/>
+</signal>
 </signals>

Commit message: forgot to save last time
Other:
- board size 160 x 100 mm -> 194.3 x 92.4 mm
Changed lines of the file:
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@@
 <board>
 <plain>
-<wire x1="0" y1="0" x2="160" y2="0" width="0" layer="20"/>
-<wire x1="160" y1="0" x2="160" y2="100" width="0" layer="20"/>
-<wire x1="160" y1="100" x2="0" y2="100" width="0" layer="20"/>
-<wire x1="0" y1="100" x2="0" y2="0" width="0" layer="20"/>
+<wire x1="0" y1="0" x2="194.29" y2="0" width="0" layer="20"/>
+<wire x1="194.29" y1="0" x2="194.29" y2="92.38" width="0" layer="20"/>
+<wire x1="194.29" y1="92.38" x2="0" y2="92.38" width="0" layer="20"/>
+<wire x1="0" y1="92.38" x2="0" y2="0" width="0" layer="20"/>
 <text x="7.4" y="15.897" size="1.27" layer="21" ratio="12" rot="R90" align="center">BNO055</text>
 <text x="13.424" y="8.001" size="0.8128" layer="21" ratio="12" align="center">Vin</text>

Commit message: added XT60 connector
Parts:
- added U$5: XT60, XT60:XT60
- moved U$1 47.2 mm to (-2.54, 47.0)
Connections:
- net GND: now also U$5.-
- net V_BATT: now also U$5.+
Other:
- board size 194.3 x 92.4 mm -> 194.3 x 81 mm
Changed lines of the file:
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@@
 <plain>
 <wire x1="0" y1="0" x2="194.29" y2="0" width="0" layer="20"/>
-<wire x1="194.29" y1="0" x2="194.29" y2="92.38" width="0" layer="20"/>
-<wire x1="194.29" y1="92.38" x2="0" y2="92.38" width="0" layer="20"/>
-<wire x1="0" y1="92.38" x2="0" y2="0" width="0" layer="20"/>
+<wire x1="194.29" y1="0" x2="194.29" y2="80.95" width="0" layer="20"/>
+<wire x1="194.29" y1="80.95" x2="0" y2="80.95" width="0" layer="20"/>
+<wire x1="0" y1="80.95" x2="0" y2="0" width="0" layer="20"/>
 <text x="7.4" y="15.897" size="1.27" layer="21" ratio="12" rot="R90" align="center">BNO055</text>
 <text x="13.424" y="8.001" size="0.8128" layer="21" ratio="12" align="center">Vin</text>
@@
 <attribute name="VALUE" x="-58.42" y="95.504" size="1.27" layer="27" ratio="10"/>
 </element>
-<element name="U$1" library="Teensy356" package="TEENSY_3.5/3.6" value="TEENSY_3.5/3.6" x="-45.72" y="66.04" smashed="yes"/>
+<element name="U$1" library="Teensy356" package="TEENSY_3.5/3.6" value="TEENSY_3.5/3.6" x="-2.54" y="46.99" smashed="yes"/>
 <element name="XB1" library="maxstream" library_urn="urn:adsk.eagle:library:270" package="XBEE-PRO" package3d_urn="urn:adsk.eagle:package:18008/1" value="XBEE-PRO" x="-25.4" y="20.32" smashed="yes">
 <attribute name="MF" value="" x="0" y="0" size="1.778" layer="27" display="off"/>
@@
 <attribute name="VALUE" x="-84.455" y="-45.1358" size="1.27" layer="27" ratio="10"/>
 </element>
+<element name="U$5" library="XT60" package="XT60" value="XT60" x="-87.63" y="-50.8" smashed="yes"/>
 </elements>
 <signals>
@@
 <contactref element="LED2" pad="K"/>
 <contactref element="LED3" pad="K"/>
+<contactref element="U$5" pad="-"/>
+<wire x1="-76.2" y1="-44.45" x2="-76.13" y2="-50.8" width="0" layer="19" extent="1-1"/>
 <wire x1="-83.82" y1="-31.75" x2="-76.2" y2="-44.45" width="0" layer="19" extent="1-1"/>
 <wire x1="-83.82" y1="-26.67" x2="-83.82" y2="-31.75" width="0" layer="19" extent="1-1"/>
@@
 <wire x1="-45.72" y1="2.54" x2="-62.23" y2="2.54" width="0" layer="19" extent="1-1"/>
 <wire x1="-36.4" y1="11.32" x2="-45.72" y2="2.54" width="0" layer="19" extent="1-1"/>
+<wire x1="-30.48" y1="39.37" x2="-36.4" y2="11.32" width="0" layer="19" extent="1-1"/>
 <wire x1="18.415" y1="6.35" x2="-36.4" y2="11.32" width="0" layer="19" extent="1-1"/>
 <wire x1="47.625" y1="7.62" x2="18.415" y2="6.35" width="0" layer="19" extent="1-1"/>
 <wire x1="57.15" y1="32.512" x2="47.625" y2="7.62" width="0" layer="19" extent="1-1"/>
-<wire x1="-73.66" y1="58.42" x2="-62.23" y2="2.54" width="0" layer="19" extent="1-1"/>
-<wire x1="-77.47" y1="80.01" x2="-73.66" y2="58.42" width="0" layer="19" extent="1-1"/>
+<wire x1="-21.59" y1="96.52" x2="-30.48" y2="39.37" width="0" layer="19" extent="1-1"/>
+<wire x1="-15.24" y1="96.52" x2="-21.59" y2="96.52" width="0" layer="19" extent="1-1"/>
+<wire x1="-59.69" y1="106.68" x2="-21.59" y2="96.52" width="0" layer="19" extent="1-1"/>
+<wire x1="-62.23" y1="95.25" x2="-59.69" y2="106.68" width="0" layer="19" extent="1-1"/>
+<wire x1="-67.31" y1="95.25" x2="-62.23" y2="95.25" width="0" layer="19" extent="1-1"/>
+<wire x1="-72.39" y1="95.25" x2="-67.31" y2="95.25" width="0" layer="19" extent="1-1"/>
+<wire x1="-77.47" y1="95.25" x2="-72.39" y2="95.25" width="0" layer="19" extent="1-1"/>
+<wire x1="-77.47" y1="80.01" x2="-77.47" y2="95.25" width="0" layer="19" extent="1-1"/>
 <wire x1="-83.82" y1="80.01" x2="-77.47" y2="80.01" width="0" layer="19" extent="1-1"/>
-<wire x1="-77.47" y1="95.25" x2="-77.47" y2="80.01" width="0" layer="19" extent="1-1"/>
-<wire x1="-72.39" y1="95.25" x2="-77.47" y2="95.25" width="0" layer="19" extent="1-1"/>
-<wire x1="-67.31" y1="95.25" x2="-72.39" y2="95.25" width="0" layer="19" extent="1-1"/>
-<wire x1="-62.23" y1="95.25" x2="-67.31" y2="95.25" width="0" layer="19" extent="1-1"/>
-<wire x1="-59.69" y1="106.68" x2="-62.23" y2="95.25" width="0" layer="19" extent="1-1"/>
-<wire x1="-21.59" y1="96.52" x2="-59.69" y2="106.68" width="0" layer="19" extent="1-1"/>
-<wire x1="-15.24" y1="96.52" x2="-21.59" y2="96.52" width="0" layer="19" extent="1-1"/>
 </signal>
 <signal name="ENABLE">
@@
 <contactref element="U$1" pad="9/CS"/>
 <contactref element="JP4" pad="5"/>
-<wire x1="-48.26" y1="58.42" x2="52.07" y2="32.512" width="0" layer="19" extent="1-1"/>
+<wire x1="-5.08" y1="39.37" x2="52.07" y2="32.512" width="0" layer="19" extent="1-1"/>
 </signal>
 <signal name="RX">
 <contactref element="U$1" pad="10/CS"/>
 <contactref element="JP4" pad="4"/>
-<wire x1="-45.72" y1="58.42" x2="54.61" y2="32.512" width="0" layer="19" extent="1-1"/>
+<wire x1="-2.54" y1="39.37" x2="54.61" y2="32.512" width="0" layer="19" extent="1-1"/>
 </signal>
 <signal name="1PPS">
@@
 <contactref element="XB1" pad="3"/>
 <contactref element="U$1" pad="1/TX"/>
-<wire x1="-68.58" y1="58.42" x2="-36.4" y2="25.32" width="0" layer="19" extent="1-1"/>
+<wire x1="-25.4" y1="39.37" x2="-36.4" y2="25.32" width="0" layer="19" extent="1-1"/>
 </signal>
 <signal name="PS1_3V">
@@
 <contactref element="JP7" pad="2"/>
 <contactref element="JP2" pad="1"/>
-<wire x1="-73.66" y1="73.66" x2="-24.13" y2="96.52" width="0" layer="19" extent="1-1"/>
-<wire x1="-36.4" y1="29.32" x2="-73.66" y2="73.66" width="0" layer="19" extent="1-1"/>
+<wire x1="-30.48" y1="54.61" x2="-24.13" y2="96.52" width="0" layer="19" extent="1-1"/>
+<wire x1="-36.4" y1="29.32" x2="-30.48" y2="54.61" width="0" layer="19" extent="1-1"/>
 <wire x1="-43.18" y1="2.54" x2="-36.4" y2="29.32" width="0" layer="19" extent="1-1"/>
 <wire x1="15.875" y1="6.35" x2="-36.4" y2="29.32" width="0" layer="19" extent="1-1"/>
@@
 <contactref element="R1" pad="2"/>
 <contactref element="R20" pad="1"/>
+<contactref element="U$5" pad="+"/>
+<wire x1="-76.2" y1="-38.1" x2="-83.13" y2="-50.8" width="0" layer="19" extent="1-1"/>
 <wire x1="-64.77" y1="2.54" x2="-76.2" y2="-38.1" width="0" layer="19" extent="1-1"/>
 <wire x1="-80.01" y1="80.01" x2="-64.77" y2="2.54" width="0" layer="19" extent="1-1"/>
@@
 <contactref element="U$1" pad="A10"/>
 <wire x1="-54.61" y1="93.98" x2="-62.23" y2="106.68" width="0" layer="19" extent="1-1"/>
-<wire x1="-63.5" y1="71.12" x2="-54.61" y2="93.98" width="0" layer="19" extent="1-1"/>
+<wire x1="-20.32" y1="52.07" x2="-54.61" y2="93.98" width="0" layer="19" extent="1-1"/>
 </signal>
 <signal name="SDI/SDA">
@@
 <contactref element="JP7" pad="4"/>
 <wire x1="20.955" y1="6.35" x2="55.245" y2="7.62" width="0" layer="19" extent="1-1"/>
-<wire x1="-53.34" y1="73.66" x2="20.955" y2="6.35" width="0" layer="19" extent="1-1"/>
+<wire x1="-10.16" y1="54.61" x2="20.955" y2="6.35" width="0" layer="19" extent="1-1"/>
 </signal>
 <signal name="SCK/SCL">
@@
 <contactref element="JP7" pad="5"/>
 <wire x1="23.495" y1="6.35" x2="50.165" y2="7.62" width="0" layer="19" extent="1-1"/>
-<wire x1="-55.88" y1="73.66" x2="23.495" y2="6.35" width="0" layer="19" extent="1-1"/>
+<wire x1="-12.7" y1="54.61" x2="23.495" y2="6.35" width="0" layer="19" extent="1-1"/>
 </signal>
 <signal name="N$3">
@@
 <contactref element="R5" pad="1"/>
 <contactref element="U$1" pad="30"/>
-<wire x1="-20.32" y1="58.42" x2="-86.36" y2="-17.78" width="0" layer="19" extent="1-1"/>
+<wire x1="22.86" y1="39.37" x2="-86.36" y2="-17.78" width="0" layer="19" extent="1-1"/>
 </signal>
 <signal name="N$16">
 <contactref element="U$1" pad="29"/>
 <contactref element="R4" pad="1"/>
-<wire x1="-22.86" y1="58.42" x2="-86.36" y2="-11.43" width="0" layer="19" extent="1-1"/>
+<wire x1="20.32" y1="39.37" x2="-86.36" y2="-11.43" width="0" layer="19" extent="1-1"/>
 </signal>
 <signal name="N$17">
 <contactref element="R3" pad="1"/>
 <contactref element="U$1" pad="28"/>
-<wire x1="-25.4" y1="58.42" x2="-86.36" y2="-5.08" width="0" layer="19" extent="1-1"/>
+<wire x1="17.78" y1="39.37" x2="-86.36" y2="-5.08" width="0" layer="19" extent="1-1"/>
 </signal>
 <signal name="N$18">
@@
 <contactref element="U$1" pad="2"/>
 <wire x1="-86.36" y1="-38.1" x2="-86.36" y2="-44.45" width="0" layer="19" extent="1-1"/>
-<wire x1="-66.04" y1="58.42" x2="-86.36" y2="-38.1" width="0" layer="19" extent="1-1"/>
+<wire x1="-22.86" y1="39.37" x2="-86.36" y2="-38.1" width="0" layer="19" extent="1-1"/>
 </signal>
 <signal name="N$1">
 <contactref element="XB1" pad="2"/>
 <contactref element="U$1" pad="0/RX"/>
-<wire x1="-36.4" y1="27.32" x2="-71.12" y2="58.42" width="0" layer="19" extent="1-1"/>
+<wire x1="-27.94" y1="39.37" x2="-36.4" y2="27.32" width="0" layer="19" extent="1-1"/>
 </signal>
 <signal name="N$2">
@@
 <contactref element="R13" pad="2"/>
 <contactref element="U$1" pad="15/A1"/>
-<wire x1="-45.72" y1="73.66" x2="-50.37" y2="81.28" width="0" layer="19" extent="1-1"/>
+<wire x1="-50.37" y1="81.28" x2="-2.54" y2="54.61" width="0" layer="19" extent="1-1"/>
 <wire x1="-64.77" y1="95.25" x2="-50.37" y2="81.28" width="0" layer="19" extent="1-1"/>
 </signal>
@@
 <contactref element="R12" pad="2"/>
 <contactref element="U$1" pad="14/A0"/>
-<wire x1="-43.18" y1="73.66" x2="-40.21" y2="81.28" width="0" layer="19" extent="1-1"/>
+<wire x1="-40.21" y1="81.28" x2="0" y2="54.61" width="0" layer="19" extent="1-1"/>
 <wire x1="-59.69" y1="95.25" x2="-40.21" y2="81.28" width="0" layer="19" extent="1-1"/>
 </signal>
@@
 <contactref element="R14" pad="2"/>
 <contactref element="U$1" pad="16/A2"/>
-<wire x1="-60.53" y1="81.28" x2="-69.85" y2="95.25" width="0" layer="19" extent="1-1"/>
-<wire x1="-48.26" y1="73.66" x2="-60.53" y2="81.28" width="0" layer="19" extent="1-1"/>
+<wire x1="-60.53" y1="81.28" x2="-5.08" y2="54.61" width="0" layer="19" extent="1-1"/>
+<wire x1="-69.85" y1="95.25" x2="-60.53" y2="81.28" width="0" layer="19" extent="1-1"/>
 </signal>
 <signal name="N$19">
@@
 <contactref element="R15" pad="2"/>
 <contactref element="U$1" pad="17/A3"/>
-<wire x1="-70.69" y1="81.28" x2="-50.8" y2="73.66" width="0" layer="19" extent="1-1"/>
+<wire x1="-70.69" y1="81.28" x2="-7.62" y2="54.61" width="0" layer="19" extent="1-1"/>
 <wire x1="-74.93" y1="95.25" x2="-70.69" y2="81.28" width="0" layer="19" extent="1-1"/>
 </signal>

Commit message: started power routing
Parts:
- moved LED1 178.0 mm to (85.1, 30.5)
- moved LED2 178.0 mm to (85.1, 25.4)
- moved LED3 178.0 mm to (85.1, 20.3)
- moved R1 178.0 mm to (88.9, 14.0)
- moved R2 178.0 mm to (88.9, 7.62)
- moved R3 178.0 mm to (88.9, 47.0)
- moved R4 178.0 mm to (88.9, 40.6)
- moved R5 178.0 mm to (88.9, 34.3)
- moved JP7 159.2 mm to (175.9, 36.8)
- moved JP8 159.2 mm to (175.9, 54.6)
- moved XB1 122.1 mm to (85.1, 72.4)
- moved C11 117.7 mm to (14.0, 16.5)
- moved R13 115.6 mm to (49.5, 97.8)
- moved R14 115.6 mm to (44.5, 97.8)
- moved PH1 115.6 mm to (73.7, 83.8)
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Routing:
- net GND: track 0.00 -> 71.7 mm
- net +5V: track 0.00 -> 46.0 mm
- net V_BATT: track 0.00 -> 17.1 mm
Other:
- board size 194.3 x 81 mm -> 194.3 x 73.3 mm
